File: PCB/DeskHub.kicad_pcb (KiCad board)
At the start: 2 copper layers, 6.6 x 6.7 mm, 120 parts, among them J1 USB_A, J2 5V Barrel, J4 USB_A, J5 USB_A, J6 USB_A, J7 USB_A, U1 TUSB4041I, U2 3.3V Reg, U3 1.1V Reg, U4 TPS2001CDGNR, U5 TPS2001CDGNR, U6 TPS2001CDGNR, U7 TPS2001CDGNR, Y1 ECS-240-20-30B-TR

Commit message: begin work on pcb placement... pray for me
Parts:
- moved J4 87.7 mm to (180.5, 135.5)
- moved J5 64.9 mm to (154.5, 135.5)
- moved C48 45.6 mm to (220.2, 93.4)
- moved C49 45.6 mm to (220.2, 95.4)
- moved C50 45.6 mm to (216.3, 89.5)
- moved C51 45.6 mm to (207.9, 93.4)
- moved C52 45.6 mm to (207.9, 95.4)
- moved C53 45.6 mm to (204.0, 89.5)
- moved C54 45.6 mm to (207.9, 107.2)
- moved C55 45.6 mm to (207.9, 109.2)
- moved C56 45.6 mm to (204.0, 103.3)
- moved C57 45.6 mm to (220.2, 107.2)
- moved C58 45.6 mm to (220.2, 109.2)
- moved C59 45.6 mm to (216.3, 103.3)
- moved R11 45.6 mm to (220.2, 97.4)
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Routing:
- added copper zone on In1.Cu, net Earth
Other:
- board size 6.6 x 6.7 mm -> 196.5 x 134.5 mm
- copper layers 2 -> 4

Commit message: organized bypass caps into groups
Parts:
- C10, C11, C12, C18, C19, C2, C20, C21, C23, C24, C25, C26, C27, C28, C29, C3, C30, C31, C32, C33, C34, C35, C36, C37, C38, C39, C4, C40, C41, C5, C6, C7, C8, C9: moved to B.Cu
- C22: footprint Capacitor_SMD:C_0201_0603Metric -> Capacitor_SMD:C_1206_3216Metric; moved to B.Cu
- moved C41 195.9 mm to (-69.7, 53.0), turned to 180 degrees
- moved C34 194.3 mm to (-69.7, 48.0), turned to 180 degrees
- moved C12 189.6 mm to (-69.7, 43.5), turned to 180 degrees
- moved C40 187.8 mm to (-61.7, 53.0), turned to 180 degrees
- moved C33 186.1 mm to (-61.7, 48.0), turned to 180 degrees
- moved C21 183.2 mm to (-58.5, 114.5), turned to 180 degrees
- moved C26 182.3 mm to (-58.5, 119.5), turned to 180 degrees
- moved C11 181.4 mm to (-61.7, 43.5), turned to 180 degrees
- moved C39 179.2 mm to (-53.2, 52.5), turned to 180 degrees
- moved C32 177.4 mm to (-53.2, 48.0), turned to 180 degrees
- moved C5 176.2 mm to (-58.5, 109.5), turned to 180 degrees
- moved C25 175.4 mm to (-51.0, 119.5), turned to 180 degrees
- moved C10 172.8 mm to (-53.2, 43.5), turned to 180 degrees
- moved C38 171.5 mm to (-45.7, 52.5), turned to 180 degrees
- moved C20 171.2 mm to (-51.0, 114.5), turned to 180 degrees
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Other:
- board text added: "1.1"
- board text added: "3.3"

Commit message: routed 4041I bypass caps
Parts:
- moved C12 225.3 mm to (151.8, 85.0), turned to -90 degrees
- moved C41 224.4 mm to (152.5, 84.6), turned to -90 degrees
- moved C34 223.8 mm to (151.1, 84.6), turned to -90 degrees
- moved C11 219.5 mm to (153.9, 84.9), turned to -90 degrees
- moved C40 218.6 mm to (154.6, 84.6), turned to -90 degrees
- moved C33 218.0 mm to (153.2, 84.6), turned to -90 degrees
- moved C25 215.3 mm to (161.7, 85.7), turned to -135 degrees
- moved C10 214.3 mm to (157.1, 84.9), turned to -90 degrees
- moved C20 213.7 mm to (160.7, 84.7), turned to -135 degrees
- moved C9 213.4 mm to (162.2, 91.9)
- moved C39 213.4 mm to (157.8, 84.5), turned to -90 degrees
- moved C4 213.2 mm to (160.9, 85.5), turned to -135 degrees
- moved C32 212.7 mm to (156.4, 84.5), turned to -90 degrees
- moved C31 212.0 mm to (161.6, 92.6)
- moved C38 211.8 mm to (162.2, 93.3)
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Routing:
- net VDD1.1: track 0.00 -> 22.5 mm, vias 0 -> 7
- net VDD3.3: track 0.00 -> 20.9 mm, vias 0 -> 4
- net Earth: track 0.00 -> 19.9 mm, vias 0 -> 20
- added copper zone on B.Cu, net Earth

Commit message: route usb diffs, power for 1 usb partially complete
Parts:
- C49, C50, C72, C73, C74, FB7, R19: moved to B.Cu
- moved C48 179.8 mm to (69.0, 150.8)
- moved C49 179.3 mm to (69.0, 142.8)
- moved R11 178.2 mm to (70.2, 145.2), turned to 90 degrees
- moved C50 177.3 mm to (67.2, 137.7), turned to 90 degrees
- moved U4 176.6 mm to (66.7, 146.8), turned to 90 degrees
- moved FB4 80.7 mm to (250.2, 142.3)
- moved R18 80.7 mm to (254.2, 140.8)
- moved C69 80.7 mm to (261.1, 141.8)
- moved C70 80.7 mm to (261.1, 143.8)
- moved C71 80.7 mm to (258.1, 138.3)
- moved J6 70.9 mm to (243.3, 163.7)
- moved U5 60.6 mm to (203.8, 86.8)
- moved C66 54.6 mm to (206.1, 154.1)
- moved C67 54.6 mm to (206.1, 156.1)
- moved C68 54.6 mm to (206.1, 158.1)
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Routing:
- net USB_DN4_D+: track 0.00 -> 132.0 mm
- net USB_DN4_D-: track 0.00 -> 131.9 mm
- net USB_DN1_D+: track 0.00 -> 104.7 mm
- net USB_DN1_D-: track 0.00 -> 104.6 mm
- net USB_DN3_D+: track 0.00 -> 86.0 mm
- net USB_DN3_D-: track 0.00 -> 86.0 mm
- net USB_DN2_D-: track 0.00 -> 72.7 mm
- net USB_DN2_D+: track 0.00 -> 72.6 mm
- net Net-(J7-VBUS): track 0.00 -> 5.87 mm
- net BOARD_5V: track 0.00 -> 5.35 mm, vias 0 -> 2
- net /Port 1 Power Switch/OVERCURRENT: track 0.00 -> 3.85 mm, vias 0 -> 1
- net BOARD_3.3V: track 0.00 -> 1.27 mm, vias 0 -> 1
- net Earth: vias 20 -> 27
- net /Port 1 Power Switch/VOUT: vias 0 -> 4
- added copper zone on B.Cu, net /Port 1 Power Switch/VOUT
- added copper zone on F.Cu, net /Port 1 Power Switch/VOUT
- added copper zone on In2.Cu, net BOARD_3.3V
- added copper zone on In2.Cu, net BOARD_5V
- added copper zone on F.Cu, net Earth
- added copper zone on B.Cu, net GNDPWR
- added copper zone on In2.Cu, net VDD1.1
- added copper zone on In2.Cu, net VDD3.3
Other:
- board size 196.5 x 134.5 mm -> 248.1 x 134.5 mm

Commit message: cont. work on usb routing
Parts:
- moved U5 103.7 mm to (119.2, 146.8), turned to 90 degrees
- moved U6 66.6 mm to (172.4, 146.8), turned to 90 degrees
- moved U7 44.3 mm to (225.9, 146.8), turned to 90 degrees
- moved C63 11.6 mm to (152.4, 154.1)
- moved C64 11.6 mm to (152.4, 156.1)
- moved C65 11.6 mm to (152.4, 158.1)
Routing:
- net USB_DN4_D+: track 132.0 -> 146.9 mm
- net USB_DN4_D-: track 131.9 -> 146.9 mm
- net USB_DN3_D-: track 86.0 -> 96.5 mm
- net USB_DN3_D+: track 86.0 -> 96.6 mm
- net /Port 1 Power Switch/PWRON_EN: track 0.00 -> 1.93 mm, vias 0 -> 1
- net Earth: track 19.9 -> 21.1 mm, vias 27 -> 37
- added copper zone on F.Cu, net /Port 2 Power Switch/VOUT
- added copper zone on F.Cu, net /Port 3 Power Switch/VOUT
- added copper zone on F.Cu, net /Port 4 Power Switch/VOUT

Commit message: began power routing
Parts:
- C13, C14, C52, C53, C55, C56, C58, C59, C63, C64, C65, C66, C67, C68, C69, C70, C71, FB2, FB3, FB4, R16, R17, R18, R2, Y1: moved to B.Cu
- moved C42 179.9 mm to (248.2, 47.1), turned to 180 degrees
- moved C43 177.2 mm to (244.1, 49.2), turned to 90 degrees
- moved C44 171.6 mm to (240.0, 50.0), turned to 90 degrees
- moved C45 168.8 mm to (237.1, 49.5), turned to 90 degrees
- moved U2 164.5 mm to (242.5, 60.5), turned to -90 degrees
- moved D2 148.7 mm to (234.0, 56.6)
- moved J2 132.9 mm to (253.8, 36.4)
- moved C51 123.9 mm to (121.2, 151.0)
- moved C52 119.9 mm to (120.3, 142.7)
- moved C53 118.5 mm to (118.4, 137.7), turned to 90 degrees
- moved R12 117.5 mm to (123.3, 145.3), turned to 90 degrees
- moved R7 91.7 mm to (230.9, 56.6), turned to 180 degrees
- moved C1 86.1 mm to (151.7, 88.9)
- moved C54 72.5 mm to (174.8, 151.2)
- moved C55 66.8 mm to (173.7, 142.8)
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Routing:
- net Net-(J6-VBUS): track 0.00 -> 12.9 mm
- net Net-(J5-VBUS): track 0.00 -> 11.4 mm
- net XI: track 0.00 -> 11.1 mm, vias 0 -> 1
- net USB_DN2_D+: track 72.6 -> 81.0 mm
- net Net-(J4-VBUS): track 0.00 -> 8.40 mm
- net USB_DN2_D-: track 72.7 -> 80.9 mm
- net XO: track 0.00 -> 7.30 mm, vias 0 -> 1
- net Earth: track 21.1 -> 27.2 mm, vias 37 -> 58
- net Net-(U1-GRSTz): track 0.00 -> 5.71 mm
- net /Port 2 Power Switch/OVERCURRENT: track 0.00 -> 4.14 mm, vias 0 -> 1
- net BOARD_3.3V: track 1.27 -> 4.69 mm, vias 1 -> 18
- net /Port 4 Power Switch/OVERCURRENT: track 0.00 -> 3.29 mm, vias 0 -> 1
- net /Port 3 Power Switch/OVERCURRENT: track 0.00 -> 3.18 mm, vias 0 -> 1
- net USB_DN1_D-: track 104.6 -> 107.5 mm
- net USB_DN1_D+: track 104.7 -> 107.5 mm
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- added copper zone on B.Cu, net /Port 2 Power Switch/VOUT
- added copper zone on B.Cu, net /Port 3 Power Switch/VOUT
- added copper zone on B.Cu, net /Port 4 Power Switch/VOUT
- added copper zone on F.Cu, net BOARD_3.3V
- added copper zone on F.Cu, net BOARD_5V
Other:
- board size 248.1 x 134.5 mm -> 212.6 x 134.5 mm

Commit message: 1.1v power net
Parts:
- C46, FB5: moved to B.Cu
- moved FB5 76.5 mm to (132.4, 85.7), turned to 180 degrees
- moved C47 69.9 mm to (119.8, 89.2), turned to -90 degrees
- moved R8 60.3 mm to (113.2, 84.9), turned to -90 degrees
- moved R9 60.3 mm to (115.1, 87.8), turned to -90 degrees
- moved R10 57.3 mm to (116.8, 87.3), turned to 180 degrees
- moved J1 7.87 mm to (98.3, 27.9)
- moved U3 7.15 mm to (118.3, 83.0)
- moved C46 7.12 mm to (117.0, 77.1)
Routing:
- net BOARD_3.3V: track 4.69 -> 12.4 mm, vias 18 -> 25
- net Net-(U3-FB): track 0.00 -> 3.46 mm
- net Net-(U3-SS): track 0.00 -> 2.69 mm
- net VDD3.3: track 22.3 -> 21.2 mm
- net VDD1.1: vias 7 -> 19
- net BOARD_1.1V: vias 0 -> 12
- added copper zone on B.Cu, net BOARD_1.1V
- added copper zone on F.Cu, net BOARD_1.1V
- added copper zone on B.Cu, net BOARD_3.3V
- added copper zone on B.Cu, net VDD1.1
